Commit message: Add Domain Randomisation, TODO: FIX MIMIC JOINTS

File: source/isaaclab_tasks/isaaclab_tasks/direct/bionic_arm/assets/urdf/EZARM_SLDASM/urdf/EZARM_SLDASM.urdf (robot description, URDF)
Before this commit: robot EZARM_SLDASM, 13 links, 12 joints
Joints:
- joint palm_joint: limit lower=0 upper=3.14159 effort=100 velocity=100 -> lower=-3.14159 upper=0 effort=100 velocity=100
